Commit message: gmapping

File: ros_robotics/urdf/dd_description.xacro (robot description, xacro)
@@ -4,5 +4,14 @@
 <!--dummy-->
 <link name="dummy">
+    <visual>
+        <origin xyz="0 0 0" rpy="0 0 0" />
+        <geometry>
+            <box size="0.001 0.001 0.001" />
+        </geometry>
+    </visual>
   </link>
+  <gazebo reference="dummy">
+    <turnGravityOff>false</turnGravityOff>
+  </gazebo>
   <!-- Base Link -->
   <link name="base_link">
@@ -44,4 +53,5 @@
   </link>
   <joint name="dummy_joint" type="fixed">
+    <origin xyz="0 0 -0.2" rpy="0 0 0"/>
      <parent link="dummy"/>
      <child link="base_link"/>

Commit message: add color

File: ros_robotics/urdf/dd_description.xacro (robot description, xacro)
@@ -2,4 +2,16 @@
 <robot name="dd_robot" xmlns:xacro="http://www.ros.org/wiki/xacro">
 <xacro:property name="hokuyo_size" value="0.05" />
+  <material name="Black">
+    <color rgba="0.0 0.0 0.0 1.0"/>
+  </material>
+  <material name="Red">
+    <color rgba="0.8 0.0 0.0 1.0"/>
+  </material>
+  <material name="White">
+    <color rgba="1.0 1.0 1.0 1.0"/>
+  </material>
+  <material name="Blue">
+    <color rgba="0.0 0.0 0.8 1.0"/>
+  </material>
 <!--dummy-->
 <link name="dummy">
@@ -14,4 +26,10 @@
     <turnGravityOff>false</turnGravityOff>
   </gazebo>
+<!--dumm_joint-->
+  <joint name="dummy_joint" type="fixed">
+    <origin xyz="0 0 0.175" rpy="0 0 0"/>
+     <parent link="dummy"/>
+     <child link="base_link"/>
+  </joint>
   <!-- Base Link -->
   <link name="base_link">
@@ -21,4 +39,5 @@
           <box size="0.8 0.5 0.25"/>
       </geometry>
+      <material name="Blue" />
     </visual>
     <!-- Base collision, mass and inertia -->
@@ -33,14 +52,17 @@
       <inertia ixx="0.13" ixy="0.0" ixz="0.0" iyy="0.37" iyz="0.0" izz="0.29"/>
     </inertial>
+  </link>
     <!-- Caster -->
-    <visual name="caster">
-      <origin xyz="0.345 0 -0.125" rpy="0 0 0" />
+    <link name="caster_link">
+    <visual>
+      <origin xyz="0 0 0" rpy="0 0 0" />
       <geometry>
         <sphere radius="0.05" />
       </geometry>
+      <material name="Black" />
     </visual>
     <!-- Caster collision, mass and inertia -->
     <collision>
-      <origin xyz="0.345 0 -0.125" rpy="0 0 0" />
+      <origin xyz="0 0 0" rpy="0 0 0" />
       <geometry>
         <sphere radius="0.05" />
@@ -52,8 +74,9 @@
     </inertial>
   </link>
-  <joint name="dummy_joint" type="fixed">
-    <origin xyz="0 0 -0.2" rpy="0 0 0"/>
-     <parent link="dummy"/>
-     <child link="base_link"/>
+  <!--Caster_joint-->
+  <joint name="caster_joint" type="fixed">
+    <origin xyz="0.345 0 -0.125" rpy="0 0 0"/>
+     <parent link="base_link"/>
+     <child link="caster_link"/>
   </joint>
   <!-- Right Wheel -->
@@ -64,4 +87,5 @@
           <cylinder length="0.1" radius="0.2" />
       </geometry>
+      <material name="Black" />
     </visual>
     <!-- Right Wheel collision, mass and inertia -->
@@ -91,4 +115,5 @@
           <cylinder length="0.1" radius="0.2" />
       </geometry>
+      <material name="Black" />
     </visual>
     <!-- Left Wheel collision, mass and inertia -->
@@ -118,4 +143,5 @@
         <box size="${hokuyo_size} ${hokuyo_size} ${hokuyo_size}"/>
       </geometry>
+      <material name="White" />
     </visual>
   </link>

File: ros_robotics/urdf/dd_robot.urdf (robot description, URDF)
Before this commit: robot dd_robot, 3 links, 2 joints
Links:
- added link caster_link, mass 0.5; collision sphere radius=0.05; visual sphere radius=0.05
- added link dummy; visual box size=0.001 0.001 0.001
- added link hokuyo_link; visual box size=0.05 0.05 0.05
- link base_link: mass None -> 5; geometry collision box size=0.8 0.5 0.25; visual box size=0.8 0.5 0.25
- link left_wheel: mass None -> 0.5
- link right_wheel: mass None -> 0.5
Joints:
- added joint caster_joint: type fixed, parent base_link, child caster_link, origin xyz=0.345 0 -0.125 rpy=0 0 0
- added joint dummy_joint: type fixed, parent dummy, child base_link, origin xyz=0 0 0.175 rpy=0 0 0
- added joint hokuyo_joint: type fixed, parent base_link, child hokuyo_link, origin xyz=0.38 0 0.1375 rpy=0 0 0
- joint joint_left_wheel: origin xyz=0 0.30 0 rpy=0 0 0 -> xyz=-0.15 0.30 0.025 rpy=0 0 0
- joint joint_right_wheel: origin xyz=0 -0.30 0 rpy=0 0 0 -> xyz=-0.15 -0.30 0.025 rpy=0 0 0
